File: Schematics/Schematics.sch (KiCad schematic (older format))
At the start: 5 parts, among them P1 Conn_02x20_Odd_Even

Commit message: Schematics Lab
Parts:
- added C1, C2: 100u, symbol pspice:C
- added C3: 100u, symbol Device:CP
- added L1: 100m, symbol Device:L
- added U1, U2, U3, U4, U5: MCP3201, symbol Analog_ADC:MCP3201
- MK1, MK2, MK3, MK4: symbol Mechanical:Mounting_Hole -> Schematics-rescue:Mounting_Hole-Mechanical
Connections:
- net labels added: +3V3, 3V3_Clean, ADC1, ADC2, ADC3, ADC4, ADC5, CLK, CS
- wire segments 52 -> 83
Other:
- note added: "40 Pin rPi"
- note added: "Lab 2 Mikrofoner"
- note added: "Lab 3 Doppler"
- note added: "Pi bridge (DC LP filter)"
- note removed: "ID_SD and ID_SC PINS:\nThese pins are reserved for HAT ID EEPROM.\n\nAt boot time this I2C interface will be\ninterrogated to look for an EEPROM\nthat identifes the attached board and\nallows automagic setup of the GPIOs\n(and optionally, Linux drivers).\n\nDO NOT USE these pins for anything other\nthan attaching an I2C ID EEPROM. Leave\nunconnected if ID EEPROM not required."
