File: Schematics/Schematics.sch (KiCad schematic (older format))
At the start: 14 parts, among them P1 Conn_02x20_Odd_Even, U1 MCP3201, U2 MCP3201, U3 MCP3201, U4 MCP3201, U5 MCP3201

Commit message: Uppdate schematics
Parts:
- added C4, C7: 1n, symbol Device:C
- added C5, C8: 100n, symbol Device:C
- added C6, C9: 6u7, symbol Device:C
- added MK5, MK6, MK7: Microphone, symbol Device:Microphone
- added R1, R2, R3, R4, R5, R6, R7, R8: 15k, symbol Device:R
- added U6: K-LC6_V2, symbol TTT4280:K-LC6_V2
- added U7, U8: MCP602, symbol Amplifier_Operational:MCP602
Connections:
- net +5V: now also U6.2 (Vcc)
- net 3V3_Clean: now also R3.2, R6.2
- net GND: now also U4.3 (IN-), U5.3 (IN-), C5.1, C8.1, R4.1, R7.1, U6.4 (GND)
- net at U1.2 (IN+): now also MK5.2 (+)
- net at U1.3 (IN-): now also MK5.1 (-)
- net at U2.2 (IN+): now also MK6.2 (+)
- net at U2.3 (IN-): now also MK6.1 (-)
- net at U3.2 (IN+): now also MK7.2 (+)
- net at U3.3 (IN-): now also MK7.1 (-)
- net at U4.2 (IN+): now also C6.1, R5.1, U7.1
- net at U5.2 (IN+): now also C9.1, R8.1, U8.1
- new net: C4.1, C6.2, R5.2, U7.2 (-)
- new net: C5.2, R3.1, R4.2, U7.3 (+)
- new net: C4.2, R1.1
- new net: R1.2, U6.3 (IF_I)
- new net: C7.1, C9.2, R8.2, U8.2 (-)
- new net: C8.2, R6.1, R7.2, U8.3 (+)
- new net: C7.2, R2.1
- new net: R2.2, U6.1 (IF_Q)
- no-connect marks 0 -> 1
Other:
- note added: "BPF [3.5,23k]Hz"
- note added: "IF_I channel"
- note added: "IF_Q channel"
- note added: "TTT4280 - Lab"
- moved on the sheet: U4, U5
